Commit message: Jun1 end commit

File: src/description/urdf/r2.urdf (robot description, URDF)
Before this commit: robot r2, 13 links, 12 joints
Links:
- removed link sensor_mast
- link realsense_camera_link: geometry visual box size=0.025 0.09 0.025
- link unitree_lidar_link: geometry visual cylinder length=0.05 radius=0.03
Joints:
- removed joint sensor_mast_joint
- joint base_joint: origin xyz=0 0 ${wheel_radius + base_height/2} rpy=0 0 0 -> xyz=0 0 ${ground_clearance + base_height/2} rpy=0 0 0
- joint realsense_camera_joint: parent sensor_mast -> body_link
- joint unitree_lidar_joint: origin xyz=0 0 0.52 rpy=0 0 0 -> xyz=0 0 0.5 rpy=0 0 0; parent sensor_mast -> body_link
