Commit message: Jun6 end of day commit

File: src/robocon_description/urdf/r2.urdf (robot description, URDF)
Before this commit: robot r2, 12 links, 11 joints
Links:
- added link storage_slide; collision box size=0.02 0.5 0.15; collision box size=0.8 0.02 0.15
Joints:
- added joint storage_slide_joint: type fixed, parent body_link, child storage_slide, origin xyz=-0.05 0 0.15 rpy=0 -0.25 0
